Commit message: asd

File: arm-tutorial/arm-tutorial/elfin/elfin_description/urdf/elfin3_no_fric_no_joint_limit.urdf.xacro (robot description, xacro)
@@ -421,5 +421,5 @@
           </clip>
         </camera>
-        <plugin name="kinect_camera_controller" filename="libgazebo_ros_openni_kinect.so">
+        <plugin name="kinect_camera_controller" filename="libgazebo_ros_openni_kinect.so">ros
           <cameraName>camera</cameraName>
           <alwaysOn>true</alwaysOn>
@@ -441,3 +441,13 @@
       </sensor>
     </gazebo>
+    <joint name="optical_joint" type="fixed">
+      <origin
+      xyz="0 0 0"
+      rpy="0 0 0" />
+      <parent
+        link="camera_link" />
+      <child
+        link="optical_link" />
+    </joint>
+    <link name="optical_link"/>
 </robot>

Commit message: edistystä

File: arm-tutorial/arm-tutorial/elfin/elfin_description/urdf/elfin3_no_fric_no_joint_limit.urdf.xacro (robot description, xacro)
@@ -451,3 +451,13 @@
     </joint>
     <link name="optical_link"/>
+    <joint name="virtual_joint" type="fixed">
+      <origin
+      xyz="0 0 0"
+      rpy=" 0 0 0" />
+      <parent
+        link="optical_link" />
+      <child
+        link="camera_desired" />
+    </joint>
+    <link name="camera_desired"/>
 </robot>

Commit message: edistystä

File: arm-tutorial/arm-tutorial/elfin/elfin_description/urdf/elfin3_no_fric_no_joint_limit.urdf.xacro (robot description, xacro)
@@ -451,4 +451,5 @@
     </joint>
     <link name="optical_link"/>
+<!--
     <joint name="virtual_joint" type="fixed">
       <origin
@@ -460,4 +461,4 @@
         link="camera_desired" />
     </joint>
-    <link name="camera_desired"/>
+    <link name="camera_desired"/> -->
 </robot>
